Commit message: Minor spelling mistake

File: ridgeback/ridgeback_description/urdf/accessories.urdf.xacro (robot description, xacro)
@@ -78,5 +78,5 @@
 	  <origin xyz="0.02 0 0" rpy="0 1.57 0" />
 	  <parent link="ur10_arm_ee_link" />
-	  <child link="gripepr_link" />
+	  <child link="gripper_link" />
   </joint>
 </robot>

Commit message: More minor updates to UR10 configs

File: ridgeback/ridgeback_description/urdf/accessories.urdf.xacro (robot description, xacro)
@@ -11,5 +11,5 @@
   <xacro:include filename="$(find ridgeback_description)/urdf/accessories/sick_lms1xx_mount.urdf.xacro" />
   <xacro:include filename="$(find ridgeback_description)/urdf/accessories/hokuyo_ust-10lx_mount.urdf.xacro" />
-  <xacro:include filename="$(find ur_description)/urdf/ur5.urdf.xacro" />
+  <xacro:include filename="$(find ur_description)/urdf/ur10.urdf.xacro" />
   <!-- If enabled, generate the front HOKUYO UST-10LX LASER payload. -->
   <xacro:if value="$(optenv RIDGEBACK_FRONT_HOKUYO_LASER 0)">
@@ -54,10 +54,10 @@
   </joint>
 <!-- Spawn arm -->
-  <xacro:ur5_robot prefix="ur10_arm_" joint_limited="true"/>
+  <xacro:ur10_robot prefix="ur10_arm_" joint_limited="true"/>
   <!-- Join arm -->
   <joint name="ur10_arm_base" type="fixed">
 	<parent link="mid_mount" />
 	<child link="ur10_arm_base_link" />
-	<origin xyz="0.22 0.0 0.0" rpy="0.0 0.0 -1.5708" />
+	<origin xyz="0.22 0.0 0.50" rpy="0.0 0.0 -1.5708" />
   </joint>
   <!-- Gripper -->

Commit message: Changed naming, removed robotiq parts

File: ridgeback/ridgeback_description/urdf/accessories.urdf.xacro (robot description, xacro)
@@ -13,5 +13,5 @@
   <xacro:include filename="$(find ur_description)/urdf/ur10.urdf.xacro" />
   <!-- If enabled, generate the front HOKUYO UST-10LX LASER payload. -->
-  <xacro:if value="$(optenv RIDGEBACK_FRONT_HOKUYO_LASER 0)">
+  <xacro:if value="$(optenv RIDGEBACK_FRONT_HOKUYO_LASER 1)">
     <xacro:hokuyo_ust-10lx_mount prefix="front"
                             topic="front/scan"
@@ -19,5 +19,5 @@
   </xacro:if>
   <!-- If enabled, generate the rear HOKUYO UST-10LX LASER payload. -->
-  <xacro:if value="$(optenv RIDGEBACK_REAR_HOKUYO_LASER 0)">
+  <xacro:if value="$(optenv RIDGEBACK_REAR_HOKUYO_LASER 1)">
     <xacro:hokuyo_ust-10lx_mount prefix="rear"
                             topic="rear/scan"
@@ -36,20 +36,20 @@
                             location="-1" />
   </xacro:if>
-  <link name="arch_link">
+  <link name="pgc02_link">
 		<visual>
 			<geometry>
-				<mesh filename="package://ridgeback_description/meshes/epfl_arch.dae" />
+				<mesh filename="package://ridgeback_description/meshes/pgc02_top.dae" />
 			</geometry>
 		</visual>
 		<collision>
 			<geometry>
-				<mesh filename="package://ridgeback_description/meshes/epfl_arch.dae" />
+				<mesh filename="package://ridgeback_description/meshes/pgc02_top.dae" />
 			</geometry>
 		</collision>
    </link>
-  <joint name="arch_joint" type="fixed">
+  <joint name="pgc02_joint" type="fixed">
 	  <origin xyz="-0.38 0 0.278" rpy="0 0 1.5" />
 	  <parent link="top_link" />
-	  <child link="arch_link" />
+	  <child link="pgc02_link" />
   </joint>
 <!-- Spawn arm -->

Commit message: fixed gripper mount

File: ridgeback/ridgeback_description/urdf/accessories.urdf.xacro (robot description, xacro)
@@ -76,5 +76,5 @@
    </link>
   <joint name="gripper_joint" type="fixed">
-	  <origin xyz="0.02 0 0" rpy="0 1.57 0" />
+	  <origin xyz="0.01 0 0" rpy="0 0 0" />
 	  <parent link="ur10_arm_ee_link" />
 	  <child link="gripper_link" />

Commit message: Gripper... GRRR

File: ridgeback/ridgeback_description/urdf/accessories.urdf.xacro (robot description, xacro)
@@ -76,5 +76,5 @@
    </link>
   <joint name="gripper_joint" type="fixed">
-	  <origin xyz="0.01 0 0" rpy="0 0 0" />
+	  <origin xyz="0.01 0 0" rpy="1.571 1.571 0" />
 	  <parent link="ur10_arm_ee_link" />
 	  <child link="gripper_link" />

Commit message: ..

File: ridgeback/ridgeback_description/urdf/accessories.urdf.xacro (robot description, xacro)
@@ -76,5 +76,5 @@
    </link>
   <joint name="gripper_joint" type="fixed">
-	  <origin xyz="0.01 0 0" rpy="1.571 1.571 0" />
+	  <origin xyz="0.01 0.0 0.0" rpy="0.0 1.571 1.571" />
 	  <parent link="ur10_arm_ee_link" />
 	  <child link="gripper_link" />

Commit message: minor mod

File: ridgeback/ridgeback_description/urdf/accessories.urdf.xacro (robot description, xacro)
@@ -65,5 +65,5 @@
 		<visual>
 			<geometry>
-				<box size="0.13 0.09 0.01" />
+				<box size="0.09 0.13 0.01" />
 			</geometry>
 			<material name="light_grey"/>
@@ -76,5 +76,5 @@
    </link>
   <joint name="gripper_joint" type="fixed">
-	  <origin xyz="0.01 0.0 0.0" rpy="0.0 1.571 1.571" />
+	  <origin xyz="0.005 0.0 0.0" rpy="0.0 1.571 0.0" />
 	  <parent link="ur10_arm_ee_link" />
 	  <child link="gripper_link" />

Commit message: Slight tweak to arm position in URDF file

File: ridgeback/ridgeback_description/urdf/accessories.urdf.xacro (robot description, xacro)
@@ -49,5 +49,5 @@
    </link>
   <joint name="pgc02_joint" type="fixed">
-	  <origin xyz="-0.38 0 0.278" rpy="0 0 1.5" />
+	  <origin xyz="0 0 0.278" rpy="0 0 1.571" />
 	  <parent link="top_link" />
 	  <child link="pgc02_link" />
@@ -59,5 +59,5 @@
 	<parent link="mid_mount" />
 	<child link="ur10_arm_base_link" />
-	<origin xyz="0.22 0.0 0.50" rpy="0.0 0.0 -1.5708" />
+	<origin xyz="0.28 0.0 0.50" rpy="0.0 0.0 -1.5708" />
   </joint>
   <!-- Gripper -->
